File: USB_CAN_CONVERTER_BASIC.sch (KiCad schematic (older format))
At the start: 22 parts, among them P1 CONN_01X05, P2 CONN_01X02, P3 USB_A, P4 CONN_01X04, U1 STM32F042C6Ux, U2 PESD2CAN, U3 TCAN332, U4 MCP1700T-3302E/TT, U5 USBLC6-2SC6

Commit message: Gerber update
Gerber update
Parts:
- removed GS3: GS2, Connect:GS2, symbol GS2
- C2, C3, C4, C5, C7, C8: footprint Resistors_SMD:R_0805 -> Capacitors_SMD:C_0805
- R4: footprint Resistors_SMD:R_0805 -> Resistors_SMD:R_0603
- U3: value TCAN332 -> TCAN332/TJA1050T; 1st Disrtib Link http://pl.farnell.com/texas-instruments/tcan332dr/can-trans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 -> http://www.tme.eu/pl/details/tja1050t_cm/uklady-scalone-int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; 1st Disrtib PN Farnell -> tme; MFG TI -> NXP; MFG Part Num TCAN332DR -> TJA1050T/CM
- U4: 1st Disrtib Link http://pl.farnell.com/microchip/mcp1700t-3302e-tt/ic-v-reg-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 -> http://www.tme.eu/pl/details/mcp1700t3302ett/stabilizatory-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; 1st Disrtib PN Farnell -> TME; 2nd Distrib Link (none) -> http://pl.farnell.com/microchip/mcp1700t-3302e-tt/ic-v-reg-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
Connections:
- net +3V3: no longer C2.1, C3.1, U3.3 (Vcc)
- net +5V: now also C2.1, C3.1, U3.3 (Vcc)
Changed lines of the file:
@@
 F 0 "C4" H 9215 1746 50  0000 L CNN
 F 1 "10n" H 9215 1655 50  0000 L CNN
-F 2 "Resistors_SMD:R_0805" H 9138 1550 50  0001 C CNN
+F 2 "Capacitors_SMD:C_0805" H 9138 1550 50  0001 C CNN
 F 3 "" H 9100 1700 50  0000 C CNN
 F 4 "08053C103KAT2A" H 9100 1700 60  0001 C CNN "MFG Part Num"
@@
 F 0 "C5" H 9615 1746 50  0000 L CNN
 F 1 "100n" H 9615 1655 50  0000 L CNN
-F 2 "Resistors_SMD:R_0805" H 9538 1550 50  0001 C CNN
+F 2 "Capacitors_SMD:C_0805" H 9538 1550 50  0001 C CNN
 F 3 "" H 9500 1700 50  0000 C CNN
 F 4 "C0805C104K3RAC" H 9500 1700 60  0001 C CNN "MFG Part Num"
@@
 F 0 "C8" H 10665 2846 50  0000 L CNN
 F 1 "1u" H 10665 2755 50  0000 L CNN
-F 2 "Resistors_SMD:R_0805" H 10588 2650 50  0001 C CNN
+F 2 "Capacitors_SMD:C_0805" H 10588 2650 50  0001 C CNN
 F 3 "" H 10550 2800 50  0000 C CNN
 F 4 "08053G105ZAT2A" H 10550 2800 60  0001 C CNN "MFG Part Num"
@@
 F 0 "C7" H 9550 2850 50  0000 L CNN
 F 1 "1u" H 9500 2750 50  0000 L CNN
-F 2 "Resistors_SMD:R_0805" H 9788 2650 50  0001 C CNN
+F 2 "Capacitors_SMD:C_0805" H 9788 2650 50  0001 C CNN
 F 3 "" H 9750 2800 50  0000 C CNN
 F 4 "08053G105ZAT2A" H 9750 2800 60  0001 C CNN "MFG Part Num"
@@
 F 4 "MCP1700T-3302E/TT" H 10150 2700 60  0001 C CNN "MFG Part Num"
 F 5 "MICROCHIP" H 10150 2700 60  0001 C CNN "MFG"
-F 6 "http://pl.farnell.com/microchip/mcp1700t-3302e-tt/ic-v-reg-ldo-250ma-smd-sot-23/dp/1296592?CMP=GRHB-FINDCHIPS" H 10150 2700 60  0001 C CNN "1st Disrtib Link"
-F 7 "Farnell" H 10150 2700 60  0001 C CNN "1st Disrtib PN"
+F 6 "http://www.tme.eu/pl/details/mcp1700t3302ett/stabilizatory-napiecia-nieregulowane-ldo/microchip-technology/mcp1700t-3302ett/" H 10150 2700 60  0001 C CNN "1st Disrtib Link"
+F 7 "TME" H 10150 2700 60  0001 C CNN "1st Disrtib PN"
+F 8 "http://pl.farnell.com/microchip/mcp1700t-3302e-tt/ic-v-reg-ldo-250ma-smd-sot-23/dp/1296592?CMP=GRHB-FINDCHIPS" H 10150 2700 60  0001 C CNN "2nd Distrib Link"
 	1    10150 2700
 	1    0    0    -1
@@
 P 3150 6150
 F 0 "U3" H 3150 6587 60  0000 C CNN
-F 1 "TCAN332" H 3150 6481 60  0000 C CNN
+F 1 "TCAN332/TJA1050T" H 3150 6481 60  0000 C CNN
 F 2 "SO:SO" H 3150 6481 60  0001 C CNN
 F 3 "" H 3000 6050 60  0000 C CNN
-F 4 "TCAN332DR" H 3150 6150 60  0001 C CNN "MFG Part Num"
-F 5 "TI" H 3150 6150 60  0001 C CNN "MFG"
-F 6 "http://pl.farnell.com/texas-instruments/tcan332dr/can-transceiver-5mbps-soic-8/dp/2526582?CMP=GRHB-FINDCHIPS" H 3150 6150 60  0001 C CNN "1st Disrtib Link"
-F 7 "Farnell" H 3150 6150 60  0001 C CNN "1st Disrtib PN"
+F 4 "TJA1050T/CM" H 3150 6150 60  0001 C CNN "MFG Part Num"
+F 5 "NXP" H 3150 6150 60  0001 C CNN "MFG"
+F 6 "http://www.tme.eu/pl/details/tja1050t_cm/uklady-scalone-interfejs-can/nxp/" H 3150 6150 60  0001 C CNN "1st Disrtib Link"
+F 7 "tme" H 3150 6150 60  0001 C CNN "1st Disrtib PN"
 	1    3150 6150
 	-1   0    0    1
 $EndComp
 $Comp
-L +3.3V #PWR014
-U 1 1 5708A6C5
-P 4750 6100
-F 0 "#PWR014" H 4750 5950 50  0001 C CNN
-F 1 "+3.3V" H 4768 6273 50  0000 C CNN
-F 2 "" H 4750 6100 50  0000 C CNN
-F 3 "" H 4750 6100 50  0000 C CNN
-	1    4750 6100
-	1    0    0    -1
-$EndComp
-$Comp
-L GND #PWR015
+L GND #PWR014
 U 1 1 5708A9FB
 P 4750 6400
-F 0 "#PWR015" H 4750 6150 50  0001 C CNN
+F 0 "#PWR014" H 4750 6150 50  0001 C CNN
 F 1 "GND" V 4758 6272 50  0000 R CNN
 F 2 "" H 4750 6400 50  0000 C CNN
@@
 F 0 "C3" H 4550 6250 50  0000 L CNN
 F 1 "10n" H 4600 6150 50  0000 L CNN
-F 2 "Resistors_SMD:R_0805" H 4788 6100 50  0001 C CNN
+F 2 "Capacitors_SMD:C_0805" H 4788 6100 50  0001 C CNN
 F 3 "" H 4750 6250 50  0000 C CNN
 F 4 "08053C103KAT2A" H 4750 6250 60  0001 C CNN "MFG Part Num"
@@
 F 0 "C2" H 4250 6250 50  0000 L CNN
 F 1 "100n" H 4250 6150 50  0000 L CNN
-F 2 "Resistors_SMD:R_0805" H 4488 6100 50  0001 C CNN
+F 2 "Capacitors_SMD:C_0805" H 4488 6100 50  0001 C CNN
 F 3 "" H 4450 6250 50  0000 C CNN
 F 4 "C0805C104K3RAC" H 4450 6250 60  0001 C CNN "MFG Part Num"
@@
 $EndComp
 $Comp
-L GND #PWR016
+L GND #PWR015
 U 1 1 5708B621
 P 4450 6400
-F 0 "#PWR016" H 4450 6150 50  0001 C CNN
+F 0 "#PWR015" H 4450 6150 50  0001 C CNN
 F 1 "GND" V 4458 6272 50  0000 R CNN
 F 2 "" H 4450 6400 50  0000 C CNN
@@
 $EndComp
 $Comp
-L GND #PWR017
+L GND #PWR016
 U 1 1 5708BDA5
 P 4200 6400
-F 0 "#PWR017" H 4200 6150 50  0001 C CNN
+F 0 "#PWR016" H 4200 6150 50  0001 C CNN
 F 1 "GND" V 4208 6272 50  0000 R CNN
 F 2 "" H 4200 6400 50  0000 C CNN
@@
 $EndComp
 $Comp
-L GND #PWR018
+L GND #PWR017
 U 1 1 5708D67B
 P 1450 7100
-F 0 "#PWR018" H 1450 6850 50  0001 C CNN
+F 0 "#PWR017" H 1450 6850 50  0001 C CNN
 F 1 "GND" V 1458 6972 50  0000 R CNN
 F 2 "" H 1450 7100 50  0000 C CNN
@@
 F 0 "R4" V 2000 5700 50  0000 R CNN
 F 1 "120R" V 1800 5700 50  0000 R CNN
-F 2 "Resistors_SMD:R_0805" H 1830 5741 50  0001 R CNN
+F 2 "Resistors_SMD:R_0603" H 1830 5741 50  0001 R CNN
 F 3 "" H 1900 5650 50  0000 C CNN
 F 4 "SMD0805-120R" H 1900 5650 60  0001 C CNN "MFG Part Num"
@@
 $EndComp
 $Comp
-L +5V #PWR019
+L +5V #PWR018
 U 1 1 5716787A
 P 9200 4250
-F 0 "#PWR019" H 9200 4100 50  0001 C CNN
+F 0 "#PWR018" H 9200 4100 50  0001 C CNN
 F 1 "+5V" H 9100 4350 50  0000 C CNN
 F 2 "" H 9200 4250 50  0000 C CNN
@@
 $EndComp
 $Comp
-L GND #PWR020
+L GND #PWR019
 U 1 1 57167911
 P 10300 4250
-F 0 "#PWR020" H 10300 4000 50  0001 C CNN
+F 0 "#PWR019" H 10300 4000 50  0001 C CNN
 F 1 "GND" H 10250 4300 50  0000 C CNN
 F 2 "" H 10300 4250 50  0000 C CNN
@@
 $EndComp
 $Comp
-L GND #PWR021
+L GND #PWR020
 U 1 1 571ACD79
 P 9250 3350
-F 0 "#PWR021" H 9250 3100 50  0001 C CNN
+F 0 "#PWR020" H 9250 3100 50  0001 C CNN
 F 1 "GND" H 9350 3200 50  0000 C CNN
 F 2 "" H 9250 3350 50  0000 C CNN
@@
 $EndComp
 $Comp
-L +5V #PWR022
+L +5V #PWR021
 U 1 1 571E7816
 P 9400 3350
-F 0 "#PWR022" H 9400 3200 50  0001 C CNN
+F 0 "#PWR021" H 9400 3200 50  0001 C CNN
 F 1 "+5V" H 9418 3523 50  0000 C CNN
 F 2 "" H 9400 3350 50  0000 C CNN
@@
 $EndComp
 $Comp
-L +3.3V #PWR023
+L +3.3V #PWR022
 U 1 1 57800AA2
 P 1150 2250
-F 0 "#PWR023" H 1150 2100 50  0001 C CNN
+F 0 "#PWR022" H 1150 2100 50  0001 C CNN
 F 1 "+3.3V" H 1168 2423 50  0000 C CNN
 F 2 "" H 1150 2250 50  0000 C CNN
@@
 	1    1150 2250
 	0    1    1    0
-$EndComp
-$Comp
-L GS2 GS3
-U 1 1 57838B89
-P 10400 1950
-F 0 "GS3" V 10300 1800 50  0000 L CNN
-F 1 "GS2" H 10468 1950 50  0001 L CNN
-F 2 "Connect:GS2" H 10468 1905 50  0001 L CNN
-F 3 "" H 10400 1950 50  0000 C CNN
-	1    10400 1950
-	0    1    1    0
-$EndComp
-$Comp
-L +3.3V #PWR024
-U 1 1 578399EB
-P 10200 1950
-F 0 "#PWR024" H 10200 1800 50  0001 C CNN
-F 1 "+3.3V" H 10218 2123 50  0000 C CNN
-F 2 "" H 10200 1950 50  0000 C CNN
-F 3 "" H 10200 1950 50  0000 C CNN
-	1    10200 1950
-	1    0    0    -1
-$EndComp
-$Comp
-L +5V #PWR025
-U 1 1 5783A2C6
-P 10600 1950
-F 0 "#PWR025" H 10600 1800 50  0001 C CNN
-F 1 "+5V" H 10618 2123 50  0000 C CNN
-F 2 "" H 10600 1950 50  0000 C CNN
-F 3 "" H 10600 1950 50  0000 C CNN
-	1    10600 1950
-	1    0    0    -1
 $EndComp
 Text Notes 7400 7500 0    60   ~ 0
@@
 	2100 5650 2100 6100
 Connection ~ 2100 6100
+$Comp
+L +5V #PWR023
+U 1 1 58627A69
+P 4750 6100
+F 0 "#PWR023" H 4750 5950 50  0001 C CNN
+F 1 "+5V" H 4768 6273 50  0000 C CNN
+F 2 "" H 4750 6100 50  0000 C CNN
+F 3 "" H 4750 6100 50  0000 C CNN
+	1    4750 6100
+	1    0    0    -1
+$EndComp
 $EndSCHEMATC
